File: schematics/tank-sensor.kicad_pcb (KiCad board)
At the start: 2 copper layers, 0 parts

Commit message: Update the schema
Parts:
- added D3: 1N4007, Diode_THT:D_DO-41_SOD81_P10.16mm_Horizontal, F.Cu at (133.5, 72.4)
- added U1: ESP32-C6-DevKitC-1, PCM_Espressif:ESP32-C6-DevKitC-1, F.Cu at (106.7, 78.7)
